File: 12x16-LED-Matrix.sch (KiCad schematic (older format))
At the start: 208 parts, among them J1 Conn_01x06, U1 IS31FL3733B

Commit message: Switch to 47k ISET resistor
Parts:
- R4: value 20k -> 47k; LCSC C25765 -> C25792
Changed lines of the file:
@@
 P 2300 3600
 F 0 "R4" H 2359 3646 50  0000 L CNN
-F 1 "20k" H 2359 3555 50  0000 L CNN
+F 1 "47k" H 2359 3555 50  0000 L CNN
 F 2 "Resistor_SMD:R_0402_1005Metric" H 2300 3600 50  0001 C CNN
 F 3 "~" H 2300 3600 50  0001 C CNN
 F 4 "0402" H 2300 3600 50  0001 C CNN "JLC"
-F 5 "C25765" H 2300 3600 50  0001 C CNN "LCSC"
+F 5 "C25792" H 2300 3600 50  0001 C CNN "LCSC"
 	1    2300 3600
 	1    0    0    -1

Commit message: Update components based on JLCPCB availability
Parts:
- C1, C2, C3, C7: value 0.47uF -> 470nf
- C4, C5, C6: value 0.1uF -> 100nf
- R1, R2, R3: footprint Resistor_SMD:R_0402_1005Metric -> Resistor_SMD:R_0603_1608Metric; JLC 0402 -> 0603; LCSC C25741 -> C25803
- R4: footprint Resistor_SMD:R_0402_1005Metric -> Resistor_SMD:R_0603_1608Metric; JLC 0402 -> 0603; LCSC C25792 -> C25819
Other:
- note added: "I2C address: 0x50"
Changed lines of the file:
@@
 F 0 "R4" H 2359 3646 50  0000 L CNN
 F 1 "47k" H 2359 3555 50  0000 L CNN
-F 2 "Resistor_SMD:R_0402_1005Metric" H 2300 3600 50  0001 C CNN
+F 2 "Resistor_SMD:R_0603_1608Metric" H 2300 3600 50  0001 C CNN
 F 3 "~" H 2300 3600 50  0001 C CNN
-F 4 "0402" H 2300 3600 50  0001 C CNN "JLC"
-F 5 "C25792" H 2300 3600 50  0001 C CNN "LCSC"
+F 4 "0603" H 2300 3600 50  0001 C CNN "JLC"
+F 5 "C25819" H 2300 3600 50  0001 C CNN "LCSC"
 	1    2300 3600
 	1    0    0    -1
@@
 P 2300 3050
 F 0 "C7" H 2392 3096 50  0000 L CNN
-F 1 "0.47uF" H 2392 3005 50  0000 L CNN
+F 1 "470nf" H 2392 3005 50  0000 L CNN
 F 2 "Capacitor_SMD:C_0402_1005Metric" H 2300 3050 50  0001 C CNN
 F 3 "~" H 2300 3050 50  0001 C CNN
@@
 F 0 "R2" H 1559 2796 50  0000 L CNN
 F 1 "100k" H 1559 2705 50  0000 L CNN
-F 2 "Resistor_SMD:R_0402_1005Metric" H 1500 2750 50  0001 C CNN
+F 2 "Resistor_SMD:R_0603_1608Metric" H 1500 2750 50  0001 C CNN
 F 3 "~" H 1500 2750 50  0001 C CNN
-F 4 "0402" H 1500 2750 50  0001 C CNN "JLC"
-F 5 "C25741" H 1500 2750 50  0001 C CNN "LCSC"
+F 4 "0603" H 1500 2750 50  0001 C CNN "JLC"
+F 5 "C25803" H 1500 2750 50  0001 C CNN "LCSC"
 	1    1500 2750
 	1    0    0    -1
@@
 F 0 "R3" H 1859 2796 50  0000 L CNN
 F 1 "100k" H 1859 2705 50  0000 L CNN
-F 2 "Resistor_SMD:R_0402_1005Metric" H 1800 2750 50  0001 C CNN
+F 2 "Resistor_SMD:R_0603_1608Metric" H 1800 2750 50  0001 C CNN
 F 3 "~" H 1800 2750 50  0001 C CNN
-F 4 "0402" H 1800 2750 50  0001 C CNN "JLC"
-F 5 "C25741" H 1800 2750 50  0001 C CNN "LCSC"
+F 4 "0603" H 1800 2750 50  0001 C CNN "JLC"
+F 5 "C25803" H 1800 2750 50  0001 C CNN "LCSC"
 	1    1800 2750
 	1    0    0    -1
@@
 F 0 "R1" H 1409 2146 50  0000 L CNN
 F 1 "100k" H 1409 2055 50  0000 L CNN
-F 2 "Resistor_SMD:R_0402_1005Metric" H 1350 2100 50  0001 C CNN
+F 2 "Resistor_SMD:R_0603_1608Metric" H 1350 2100 50  0001 C CNN
 F 3 "~" H 1350 2100 50  0001 C CNN
-F 4 "0402" H 1350 2100 50  0001 C CNN "JLC"
-F 5 "C25741" H 1350 2100 50  0001 C CNN "LCSC"
+F 4 "0603" H 1350 2100 50  0001 C CNN "JLC"
+F 5 "C25803" H 1350 2100 50  0001 C CNN "LCSC"
 	1    1350 2100
 	1    0    0    -1
@@
 P 1850 1750
 F 0 "C3" H 1942 1796 50  0000 L CNN
-F 1 "0.47uF" H 1942 1705 50  0000 L CNN
+F 1 "470nf" H 1942 1705 50  0000 L CNN
 F 2 "Capacitor_SMD:C_0402_1005Metric" H 1850 1750 50  0001 C CNN
 F 3 "~" H 1850 1750 50  0001 C CNN
@@
 P 2300 1750
 F 0 "C6" H 2392 1796 50  0000 L CNN
-F 1 "0.1uF" H 2392 1705 50  0000 L CNN
+F 1 "100nf" H 2392 1705 50  0000 L CNN
 F 2 "Capacitor_SMD:C_0402_1005Metric" H 2300 1750 50  0001 C CNN
 F 3 "~" H 2300 1750 50  0001 C CNN
@@
 P 1850 1400
 F 0 "C2" H 1942 1446 50  0000 L CNN
-F 1 "0.47uF" H 1942 1355 50  0000 L CNN
+F 1 "470nf" H 1942 1355 50  0000 L CNN
 F 2 "Capacitor_SMD:C_0402_1005Metric" H 1850 1400 50  0001 C CNN
 F 3 "~" H 1850 1400 50  0001 C CNN
@@
 P 2300 1400
 F 0 "C5" H 2392 1446 50  0000 L CNN
-F 1 "0.1uF" H 2392 1355 50  0000 L CNN
+F 1 "100nf" H 2392 1355 50  0000 L CNN
 F 2 "Capacitor_SMD:C_0402_1005Metric" H 2300 1400 50  0001 C CNN
 F 3 "~" H 2300 1400 50  0001 C CNN
@@
 P 1850 1100
 F 0 "C1" H 1942 1146 50  0000 L CNN
-F 1 "0.47uF" H 1942 1055 50  0000 L CNN
+F 1 "470nf" H 1942 1055 50  0000 L CNN
 F 2 "Capacitor_SMD:C_0402_1005Metric" H 1850 1100 50  0001 C CNN
 F 3 "~" H 1850 1100 50  0001 C CNN
@@
 P 2300 1100
 F 0 "C4" H 2392 1146 50  0000 L CNN
-F 1 "0.1uF" H 2392 1055 50  0000 L CNN
+F 1 "100nf" H 2392 1055 50  0000 L CNN
 F 2 "Capacitor_SMD:C_0402_1005Metric" H 2300 1100 50  0001 C CNN
 F 3 "~" H 2300 1100 50  0001 C CNN
@@
 	3250 4100 3150 4100
 Connection ~ 3150 4100
+Text Notes 3000 4250 2    50   ~ 0
+I2C address: 0x50
 $EndSCHEMATC
